File: boards/GIMIX Serial dumb/GIMIX Serial dumb/GIMIX Serial dumb.kicad_sch (KiCad schematic)
At the start: 48 parts, among them J1 RS232 Port, J2 Conn_01x13, J3 RS232 Port, J4 Conn_01x13, J5 Power, P1 SS30 Bus, U1 LM7805_TO220, U10 L7912, U2 75189, U3 MC6850_new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

Commit message: two port serial board finished finished
Other:
- company: (none) -> 100% Offner
- title: (none) -> GIMIX two port Serial board
Changed lines of the file:
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@@
 	(generator_version "9.0")
 	(paper "A4")
+	(title_block
+		(title "GIMIX two port Serial board")
+		(date "2026-06-25")
+		(rev "0.1")
+		(company "100% Offner")
+		(comment 1 "v0.1: Initial")
+	)
 	(text "INDEX PIN"
 		(exclude_from_sim no)
