File: boards/GIMIX Mainboard/GIMIX Mainboard/GIMIX Mainboard.kicad_sch (KiCad schematic)
At the start: 21 parts, among them SW1 SW_DIP_x10, SW2 SW_DIP_x10, U1 74LS640, U10 74LS136, U11 74LS136, U12 74LS00, U13 74LS121, U2 74LS240, U3 74LS240, U4 74LS240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

Commit message: new mainboard updated
Connections:
- net RST is gone; now on net ~{IORES}: U3.18 (O0a), U4.18 (O0a), U5.18 (O0a)
- net SW2-1: now also RP14.6 (R5); no longer RP14.10 (R9)
- net SW_A16: now also RP14.7 (R6); no longer RP14.6 (R5)
- net SW_A17: now also RP14.8 (R7); no longer RP14.7 (R6)
- net SW_A18: now also RP14.9 (R8); no longer RP14.8 (R7)
- net SW_A19: now also RP14.10 (R9); no longer RP14.9 (R8)
Changed lines of the file:
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@@
 		(title "GIMIX Mainboard 24-0049 ")
 		(date "2026-06-24")
-		(rev "0.1")
+		(rev "0.2")
 		(company "100% Offner")
 		(comment 1 "v0.1: Initial")
+		(comment 2 "v0.2: FIRQ to JA2 added, IORES conn.")
 	)
 	(rectangle
@@
 	)
 	(label "SW_A18"
-		(at 205.74 195.58 90)
+		(at 208.28 195.58 90)
 		(effects
 			(font
@@
 		)
 	)
-	(label "RST"
-		(at 63.5 229.87 180)
-		(effects
-			(font
-				(size 1.27 1.27)
-			)
-			(justify right bottom)
-		)
-	)
 	(label "IOD1"
 		(at 15.24 64.77 0)
@@
 	)
 	(label "SW_A19"
-		(at 208.28 195.58 90)
+		(at 210.82 195.58 90)
 		(effects
 			(font
@@
 		)
 	)
+	(label "~{IORES}"
+		(at 63.5 123.19 180)
+		(effects
+			(font
+				(size 1.27 1.27)
+			)
+			(justify right bottom)
+		)
+	)
 	(label "EXT_ON_OUT"
 		(at 195.58 203.2 180)
@@
 		)
 	)
-	(label "RST"
-		(at 63.5 123.19 180)
-		(effects
-			(font
-				(size 1.27 1.27)
-			)
-			(justify right bottom)
-		)
-	)
 	(label "A5_int"
 		(at 63.5 242.57 180)
@@
 		)
 	)
-	(label "RST"
-		(at 63.5 176.53 180)
-		(effects
-			(font
-				(size 1.27 1.27)
-			)
-			(justify right bottom)
-		)
-	)
 	(label "A5_int"
 		(at 152.4 111.76 0)
@@
 		)
 	)
+	(label "~{IORES}"
+		(at 63.5 176.53 180)
+		(effects
+			(font
+				(size 1.27 1.27)
+			)
+			(justify right bottom)
+		)
+	)
 	(label "SW_A7"
 		(at 205.74 129.54 90)
@@
 	)
 	(label "SW_A17"
-		(at 203.2 195.58 90)
+		(at 205.74 195.58 90)
 		(effects
 			(font
@@
 	)
 	(label "SW2-1"
-		(at 210.82 195.58 90)
+		(at 200.66 195.58 90)
 		(effects
 			(font
@@
 	)
 	(label "SW_A16"
-		(at 200.66 195.58 90)
+		(at 203.2 195.58 90)
 		(effects
 			(font
@@
 		)
 	)
+	(label "~{IORES}"
+		(at 63.5 229.87 180)
+		(effects
+			(font
+				(size 1.27 1.27)
+			)
+			(justify right bottom)
+		)
+	)
