File: boards/GIMIX Mainboard/GIMIX Mainboard/connectors.kicad_sch (KiCad schematic)
At the start: 54 parts, among them J1 Mainboard, P1 SS-50 Bus, P10 SS-50 Bus, P11 SS-50 Bus, P12 SS-50 Bus, P13 SS-50 Bus, P14 SS-50 Bus, P15 SS-50 Bus, P2 SS-50 Bus, P3 SS-50 Bus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

Commit message: new mainboard updated
Connections:
- net ~{FIRQ}: now also JA2.3 (Pin_3)
Changed lines of the file:
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@@
 		(title "GIMIX Mainboard 24-0049 ")
 		(date "2026-06-24")
-		(rev "0.1")
+		(rev "0.2")
 		(company "100% Offner")
 		(comment 1 "v0.1: Initial")
@@
 		(effects
 			(font
+				(size 1.27 1.27)
+			)
+			(justify left bottom)
+		)
+	)
+	(label "~{FIRQ}"
+		(at 264.16 204.47 0)
+		(effects
+			(font
