File: boards/GIMIX Mainboard/GIMIX Mainboard/connectors.kicad_sch (KiCad schematic)
At the start: 54 parts, among them J1 Mainboard, P1 SS-50 Bus, P10 SS-50 Bus, P11 SS-50 Bus, P12 SS-50 Bus, P13 SS-50 Bus, P14 SS-50 Bus, P15 SS-50 Bus, P2 SS-50 Bus, P3 SS-50 Bus, P4 SS-50 Bus, P5 SS-50 Bus, P6 SS-50 Bus, P7 SS-50 Bus, P8 SS-50 Bus, P9 SS-50 Bus

Commit message: motherboard new version silkscreen added
Parts:
- CA1: value Conn_01x05 -> 6800 Reset Conn.
- CA2: value Conn_01x04 -> Pilot Light Conn.
- J1: value Mainboard -> BaudRate Generator Board
- JA1: value Conn_02x05_Odd_Even -> 50pin to 30pinBaudrate Option
- JA2: value Conn_01x05 -> Interrupt Option
- JA5: value Conn_01x06 -> Termination Option
- renumbered IO1 to IO0, IO2 to IO1, IO3 to IO2, IO4 to IO3, IO5 to IO4, IO6 to IO5, IO7 to IO6, IO8 to IO7
Other:
- moved on the sheet: CA1
Changed lines of the file:
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@@
 		(title "GIMIX Mainboard 24-0049 ")
 		(date "2026-06-24")
-		(rev "0.2")
+		(rev "0.3")
 		(company "100% Offner")
 		(comment 1 "v0.1: Initial")
+		(comment 2 "v0.2: FIRQ to JA2 added, IORES conn.")
 	)
 	(junction
@@
 	)
 	(junction
-		(at 308.61 181.61)
+		(at 316.23 181.61)
 		(diameter 0)
 		(color 0 0 0 0)
@@
 	)
 	(no_connect
-		(at 309.88 176.53)
+		(at 317.5 176.53)
 	)
 	(no_connect
@@
 	)
 	(no_connect
-		(at 309.88 184.15)
+		(at 317.5 184.15)
 	)
 	(bus_entry
@@
 	(wire
 		(pts
-			(xy 298.45 173.99) (xy 309.88 173.99)
+			(xy 306.07 173.99) (xy 317.5 173.99)
 		)
 		(stroke
@@
 	(wire
 		(pts
-			(xy 308.61 181.61) (xy 308.61 185.42)
+			(xy 316.23 181.61) (xy 316.23 185.42)
 		)
 		(stroke
@@
 	(wire
 		(pts
-			(xy 308.61 181.61) (xy 308.61 179.07)
+			(xy 316.23 181.61) (xy 316.23 179.07)
 		)
 		(stroke
@@
 	(wire
 		(pts
-			(xy 309.88 181.61) (xy 308.61 181.61)
+			(xy 317.5 181.61) (xy 316.23 181.61)
 		)
 		(stroke
@@
 	(wire
 		(pts
-			(xy 308.61 179.07) (xy 309.88 179.07)
+			(xy 316.23 179.07) (xy 317.5 179.07)
 		)
 		(stroke
@@
 	)
 	(label "~{MRDY}"
-		(at 298.45 173.99 0)
+		(at 306.07 173.99 0)
 		(effects
 			(font
@@
 		(on_board yes)
 		(dnp no)
-		(fields_autoplaced yes)
 		(property "Reference" "JA2"
-			(at 285.75 203.1999 0)
+			(at 279.146 194.056 0)
 			(effects
 				(font
@@
 			)
 		)
-		(property "Value" "Conn_01x05"
-			(at 285.75 205.7399 0)
+		(property "Value" "Interrupt Option"
+			(at 279.146 196.596 0)
 			(effects
 				(font
@@
 		(on_board yes)
 		(dnp no)
-		(property "Reference" "IO6"
+		(property "Reference" "IO5"
 			(at 104.267 165.1 0)
 			(effects
@@
 			(project "GIMIX Mainboard"
 				(path "/471d184b-f3be-460f-9c44-6b4c4ffac74b/7c0d5175-39d7-4f8a-8889-08dc797cb17c"
-					(reference "IO6")
+					(reference "IO5")
 					(unit 1)
 				)
@@
 		(on_board yes)
 		(dnp no)
-		(property "Reference" "IO3"
+		(property "Reference" "IO2"
 			(at 66.167 165.1 0)
 			(effects
@@
 			(project "GIMIX Mainboard"
 				(path "/471d184b-f3be-460f-9c44-6b4c4ffac74b/7c0d5175-39d7-4f8a-8889-08dc797cb17c"
-					(reference "IO3")
+					(reference "IO2")
 					(unit 1)
 				)
@@
 		(on_board yes)
 		(dnp no)
-		(fields_autoplaced yes)
 		(property "Reference" "JA5"
-			(at 331.47 143.5099 0)
+			(at 326.644 132.588 0)
 			(effects
 				(font
@@
 			)
 		)
-		(property "Value" "Conn_01x06"
-			(at 331.47 146.0499 0)
+		(property "Value" "Termination Option"
+			(at 326.644 135.128 0)
 			(effects
 				(font
@@
 		(on_board yes)
 		(dnp no)
-		(property "Reference" "IO8"
+		(property "Reference" "IO7"
 			(at 129.667 165.1 0)
 			(effects
@@
 			(project "GIMIX Mainboard"
 				(path "/471d184b-f3be-460f-9c44-6b4c4ffac74b/7c0d5175-39d7-4f8a-8889-08dc797cb17c"
-					(reference "IO8")
+					(reference "IO7")
 					(unit 1)
 				)
@@
 		(on_board yes)
 		(dnp no)
-		(property "Reference" "IO7"
+		(property "Reference" "IO6"
 			(at 116.967 165.1 0)
 			(effects
@@
 			(project "GIMIX Mainboard"
 				(path "/471d184b-f3be-460f-9c44-6b4c4ffac74b/7c0d5175-39d7-4f8a-8889-08dc797cb17c"
-					(reference "IO7")
+					(reference "IO6")
 					(unit 1)
 				)
@@
 			)
 		)
-		(property "Value" "Conn_02x05_Odd_Even"
+		(property "Value" "50pin to 30pinBaudrate Option"
 			(at 274.32 135.89 0)
 			(effects
@@
 	(symbol
 		(lib_id "Connector_Generic:Conn_01x05")
-		(at 314.96 179.07 0)
+		(at 322.58 179.07 0)
 		(unit 1)
 		(exclude_from_sim no)
@@
 		(dnp no)
 		(property "Reference" "CA1"
-			(at 317.5 177.7999 0)
+			(at 319.786 168.148 0)
 			(effects
 				(font
@@
 			)
 		)
-		(property "Value" "Conn_01x05"
-			(at 317.5 180.3399 0)
+		(property "Value" "6800 Reset Conn."
+			(at 319.786 170.688 0)
 			(effects
 				(font
@@
 		)
 		(property "Footprint" "Connector_PinHeader_2.54mm:PinHeader_1x05_P2.54mm_Vertical"
-			(at 314.96 179.07 0)
+			(at 322.58 179.07 0)
 			(effects
 				(font
@@
 		)
 		(property "Datasheet" "~"
-			(at 314.96 179.07 0)
+			(at 322.58 179.07 0)
 			(effects
 				(font
@@
 		)
 		(property "Description" "Generic connector, single row, 01x05, script generated (kicad-library-utils/schlib/autogen/connector/)"
-			(at 314.96 179.07 0)
+			(at 322.58 179.07 0)
 			(effects
 				(font
@@
 		(on_board yes)
 		(dnp no)
-		(property "Reference" "IO5"
+		(property "Reference" "IO4"
 			(at 91.567 165.1 0)
 			(effects
@@
 			(project "GIMIX Mainboard"
 				(path "/471d184b-f3be-460f-9c44-6b4c4ffac74b/7c0d5175-39d7-4f8a-8889-08dc797cb17c"
-					(reference "IO5")
+					(reference "IO4")
 					(unit 1)
 				)
@@
 		(on_board yes)
 		(dnp no)
-		(property "Reference" "IO1"
+		(property "Reference" "IO0"
 			(at 40.767 165.1 0)
 			(effects
@@
 			(project "GIMIX Mainboard"
 				(path "/471d184b-f3be-460f-9c44-6b4c4ffac74b/7c0d5175-39d7-4f8a-8889-08dc797cb17c"
-					(reference "IO1")
+					(reference "IO0")
 					(unit 1)
 				)
@@
 		(on_board yes)
 		(dnp no)
-		(property "Reference" "IO2"
+		(property "Reference" "IO1"
 			(at 53.467 165.1 0)
 			(effects
@@
 			(project "GIMIX Mainboard"
 				(path "/471d184b-f3be-460f-9c44-6b4c4ffac74b/7c0d5175-39d7-4f8a-8889-08dc797cb17c"
-					(reference "IO2")
+					(reference "IO1")
 					(unit 1)
 				)
@@
 		(on_board yes)
 		(dnp no)
-		(property "Reference" "IO4"
+		(property "Reference" "IO3"
 			(at 78.867 165.1 0)
 			(effects
@@
 			(project "GIMIX Mainboard"
 				(path "/471d184b-f3be-460f-9c44-6b4c4ffac74b/7c0d5175-39d7-4f8a-8889-08dc797cb17c"
-					(reference "IO4")
+					(reference "IO3")
 					(unit 1)
 				)
@@
 	(symbol
 		(lib_id "power:GND")
-		(at 308.61 185.42 0)
+		(at 316.23 185.42 0)
 		(unit 1)
 		(exclude_from_sim no)
@@
 		(fields_autoplaced yes)
 		(property "Reference" "#PWR073"
-			(at 308.61 191.77 0)
+			(at 316.23 191.77 0)
 			(effects
 				(font
@@
 		)
 		(property "Value" "GND"
-			(at 308.61 190.5 0)
+			(at 316.23 190.5 0)
 			(effects
 				(font
@@
 		)
 		(property "Footprint" ""
-			(at 308.61 185.42 0)
+			(at 316.23 185.42 0)
 			(effects
 				(font
@@
 		)
 		(property "Datasheet" ""
-			(at 308.61 185.42 0)
+			(at 316.23 185.42 0)
 			(effects
 				(font
@@
 		)
 		(property "Description" "Power symbol creates a global label with name \"GND\" , ground"
-			(at 308.61 185.42 0)
+			(at 316.23 185.42 0)
 			(effects
 				(font
@@
 		(on_board yes)
 		(dnp no)
-		(fields_autoplaced yes)
 		(property "Reference" "CA2"
-			(at 285.75 177.7999 0)
+			(at 280.67 169.672 0)
 			(effects
 				(font
@@
 			)
 		)
-		(property "Value" "Conn_01x04"
-			(at 285.75 180.3399 0)
+		(property "Value" "Pilot Light Conn."
+			(at 280.67 172.212 0)
 			(effects
 				(font
@@
 			)
 		)
-		(property "Value" "Mainboard"
+		(property "Value" "BaudRate Generator Board"
 			(at 179.324 207.264 0)
 			(effects
