File: boards/GIMIX Mainboard/GIMIX Mainboard/GIMIX Mainboard.kicad_pcb (KiCad board)
At the start: 2 copper layers, 482.6 x 228.6 mm, 98 parts, among them J1 Mainboard, J2 Screw_Terminal_01x02, J3 Screw_Terminal_01x02, J4 Screw_Terminal_01x02, J5 Screw_Terminal_01x02, J6 Screw_Terminal_01x02, J7 Screw_Terminal_01x02, P1 SS-50 Bus, P10 SS-50 Bus, P11 SS-50 Bus, P12 SS-50 Bus, P13 SS-50 Bus, P14 SS-50 Bus, P15 SS-50 Bus, P2 SS-50 Bus, P3 SS-50 Bus, P4 SS-50 Bus, P5 SS-50 Bus, P6 SS-50 Bus, P7 SS-50 Bus, P8 SS-50 Bus, P9 SS-50 Bus, SW1 SW_DIP_x10, SW2 SW_DIP_x10, U1 74LS640, U10 74LS136, U11 74LS136, U12 74LS00, U13 74LS121, U2 74LS240, U3 74LS240, U4 74LS240, U5 74LS240, U6 LM7805_TO220, U7 74LS138, U8 74LS136, U9 74LS136

Commit message: motherboard new version silkscreen added
Parts:
- CA1: value Conn_01x05 -> 6800 Reset Conn.
- CA2: value Conn_01x04 -> Pilot Light Conn.
- J1: value Mainboard -> BaudRate Generator Board
- JA1: value Conn_02x05_Odd_Even -> 50pin to 30pinBaudrate Option
- JA2: value Conn_01x05 -> Interrupt Option
- JA3: value Jumper_3_Open -> Slow IO Option
- JA4: value Conn_01x04 -> PIO Disc Option
- JA5: value Conn_01x06 -> Termination Option
- moved RP13 0.76 mm to (449.3, 50.8)
- moved RP12 0.63 mm to (449.3, 54.0)
- renumbered IO1 to IO0, IO2 to IO1, IO3 to IO2, IO4 to IO3, IO5 to IO4, IO6 to IO5, IO7 to IO6, IO8 to IO7
Routing:
- net /IOR/~{W}: track 337.6 -> 336.4 mm
- net /~{IORES}: track 338.8 -> 337.7 mm
- net GND: track 2595.1 -> 2594.2 mm
- net +5V: track 1283.2 -> 1284.1 mm
- net /RS3: track 290.3 -> 289.6 mm
- net /RS0: track 271.2 -> 270.5 mm
- net /RS1: track 271.2 -> 270.4 mm
- net /IOE: track 393.8 -> 393.0 mm
- net /RS2: track 307.7 -> 307.1 mm
Other:
- board text added: "+5V"
- board text added: "110B"
- board text added: "1200B"
- board text added: "150B"
- board text added: "300B"
- board text added: "600B"
- board text added: "6800 RESET"
- board text added: "A16"
- board text added: "A17"
- board text added: "A18"
- board text added: "A19"
- board text added: "JA1: 50pin to 30pin Baudrate Option"
- board text added: "JA2: Interrupt Option (UD1, UD2 Connections)"
- board text added: "JA3: Slow IO Option"
- board text added: "JA4: PIO Disc Option"
- board text added: "JA5: Termination Points for ~{MRST}/MRDY and BUSY/~{NMI}"
- board text added: "Q(UD1)"
- board text added: "RS2(UD3)"
- board text added: "RS3(UD4)"
- board text added: "SW1: A19 A18 A17 A16 EXON A15 A14 A13 A12 IO Dis."
- board text added: "SW2: A11 A10 A9 A8 A7 A6 A5 IOSZ 16 IOSZ 8 IOSZ 4"
- board text added: "U11-3"
- board text added: "U2: IO Buffer"
- board text added: "U3: IO Size 4 Addresses"
- board text added: "U4: IO Size 8 Addresses"
- board text added: "U5: IO Size 16 Addresses"
- board text added: "x"
- board text added: "~{BREQ}"
- board text added: "~{FIRQ}(UD2)"
- board text added: "~{FIRQ}/~{NMI} to 30p. BUS"
- board text added: "~{IOSEL5}"
- board text added: "~{MRDY}"
- board text added: "~{MRST}/ MRDY"
- board text added: "~{NMI}"
- board text removed: "RESET"
