File: boards/GIMIX Mainboard/GIMIX Mainboard old version/connectors.kicad_sch (KiCad schematic)
At the start: 48 parts, among them J2 Conn_02x05_Counter_Clockwise, J3 Conn_02x02_Odd_Even, J4 P, J5 Screw_Terminal_01x04, J6 Screw_Terminal_01x14, P1 SS-50 Bus, P10 SS-50 Bus, P11 SS-50 Bus, P12 SS-50 Bus, P13 SS-50 Bus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

Commit message: Motherboard old version cleanup
Parts:
- added RN4: R_Network09, Resistor_THT:R_Array_SIP10, symbol Device:R_Network09
Connections:
- net GND: now also RN4.1 (common)
- net IOD0: now also RN4.2 (R1)
- net IOD1: now also RN4.3 (R2)
- net IOD2: now also RN4.4 (R3)
- net IOD3: now also RN4.5 (R4)
- net IOD4: now also RN4.6 (R5)
- net IOD5: now also RN4.7 (R6)
- net IOD6: now also RN4.8 (R7)
- net IOD7: now also RN4.9 (R8)
- no-connect marks 1 -> 2
Other:
- note added: "UD1 UD2 UD3 UD4"
