File: boards/GIMIX 6809 CPU Plus/GIMIX 6809 CPU Plus/GIMIX 6809 CPU Plus.kicad_pcb (KiCad board)
At the start: 2 copper layers, 248.9 x 139.7 mm, 165 parts, among them P1 SS-50 Bus, Q1 BC337, Q2 BC337, Q3 BC337, SW1 OPTION, SW2 CONFIG, U1 MM58167, U10 74LS04, U11 74LS161, U12 74LS161, U13 74LS123, U14 74LS74, U15 74LS00, U16 74LS32, U17 74LS136, U18 74LS20, U19 74LS32, U2 MC6840, U20 74LS12, U21 AM93L422, U22 AM93L422, U23 74LS174, U24 74LS157, U25 74LS20, U26 74LS04, U27 74LS02, U28 LM7812_TO220, U29 LM7805_TO220, U3 9511, U30 LM7805_TO220, U31 LM7905_TO220, U32 74LS30, U33 74LS240, U34 74LS367, U35 74LS136, U36 FPLA, U37 DS8T28N, U38 DS8T28N, U39 74S189, U4 27C32, U40 74S189, U41 DS8T28N, U42 DS8T28N, U43 74LS174, U44 DS8T28N, U45 DS8T28N, U46 74LS30, U47 MC6809, U48 74LS244, U49 74LS640, U5 27C32, U50 74LS640, U51 74LS00, U52 74LS00, U53 74LS74, U54 74LS04, U6 27C32, U7 27C32, U8 2114, U9 2114, Y1 32k768, Y2 16M, Y3 12M

Commit message: CPU 6809 plus update
Parts:
- D1: value ? -> 1N4001
- R1: value ? -> 100E
- R10, R14, R23, R9, RP3: value ? -> 10k
- R11, R13, R18, R4, R5, R8: value ? -> 1k
- R15, R20: value ? -> 10E
- R16, R2, R3: value ? -> 680E
- R17, R22, R27, R6: value ? -> 4k7
- R19, R21: value ? -> 22k
- U34: value 74LS367 -> 74LS368
Other:
- board text added: "Battery Footprint missing!"
- board text added: "Remake by 100% Offner 2026"
