File: boards/GIMIX 6809 CPU Plus/GIMIX 6809 CPU Plus/GIMIX 6809 CPU Plus.kicad_sch (KiCad schematic)
At the start: 27 parts, among them P1 SS-50 Bus, SW1 OPTION, SW2 CONFIG, U15 74LS00, U16 74LS32, U18 74LS20, U32 74LS30, U33 74LS240, U35 74LS136, U36 FPLA, U37 DS8T28N, U38 DS8T28N, U41 DS8T28N, U42 DS8T28N, U44 DS8T28N, U45 DS8T28N, U49 74LS640, U50 74LS640, U52 74LS00

Commit message: CPU 6809 plus update
Parts:
- R10, R23, R9: value ? -> 10k
- R16: value ? -> 680E
Other:
- note added: "check all chips. They are mostly guesswork except: U21, U22, U23, U37, U39, U40, U43, U44, U45. U8, U9, U1, U2, U3. They are mentioned in the documentation. The following ICs are written on the schematic: U38, U41, U42, The following ICs are clear too: EPROMS U4-U7, CPU: U47, FPLA: U36, Check especially: U17 74LS136 - checked U20: 74LS12 - checked Speed grade of Buffers (74LS244 or 'F244) - all L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"
- note removed: "check all chips. They are mostly guesswork except: U21, U22, U23, U37, U39, U40, U43, U44, U45. U8, U9, U1, U2, U3. They are mentioned in the documentation. The following ICs are written on the schematic: U38, U41, U42, The following ICs are clear too: EPROMS U4-U7, CPU: U47, FPLA: U36, Check especially: U17 74LS136 ? U20: 74LS12 ? Speed grade of Buffers (74LS244 or 'F244), U49, U50: both 'LS640 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"
Changed lines of the file:
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@@
 		(title "GIMIX 6809 CPU Plus")
 		(date "2026-07-02")
-		(rev "0.1")
+		(rev "0.2")
 		(company "100% Offner")
 		(comment 1 "v0.1: Initial")
+		(comment 2 "v0.2: ch. U34 -> 'LS368, ")
 	)
 	(text "from BUS"
@@
 		)
 	)
-	(text "check all chips.\nThey are mostly guesswork except:\nU21, U22, U23, U37, U39, U40, U43, U44, U45.\nU8, U9, U1, U2, U3.\nThey are mentioned in the documentation.\nThe following ICs are written on the schematic:\nU38, U41, U42,\nThe following ICs are clear too:\nEPROMS U4-U7,\nCPU: U47,\nFPLA: U36,\n\nCheck especially: \nU17 74LS136 ?\nU20: 74LS12 ?\nSpeed grade of Buffers (74LS244 or 'F244),\nU49, U50: both 'LS640 ?\nU24: 'LS157 ?\n\n\nAlso: check all the passive components,\nthey are all missing!"
+	(text "check all chips.\nThey are mostly guesswork except:\nU21, U22, U23, U37, U39, U40, U43, U44, U45.\nU8, U9, U1, U2, U3.\nThey are mentioned in the documentation.\nThe following ICs are written on the schematic:\nU38, U41, U42,\nThe following ICs are clear too:\nEPROMS U4-U7,\nCPU: U47,\nFPLA: U36,\n\nCheck especially: \nU17 74LS136 - checked\nU20: 74LS12 - checked\nSpeed grade of Buffers (74LS244 or 'F244) - all LS\nU49, U50: both 'LS640 - checked\nU24: 'LS157 - checked\n\n\nAlso: check all the passive components,\nthey are all missing!"
 		(exclude_from_sim no)
 		(at 230.886 160.02 0)
@@
 			)
 		)
-		(property "Value" "?"
+		(property "Value" "10k"
 			(at 149.86 121.9199 0)
 			(effects
@@
 			)
 		)
-		(property "Value" "?"
+		(property "Value" "10k"
 			(at 142.24 121.9199 0)
 			(effects
@@
 			)
 		)
-		(property "Value" "?"
+		(property "Value" "680E"
 			(at 219.71 172.7199 0)
 			(effects
@@
 			)
 		)
-		(property "Value" "?"
+		(property "Value" "10k"
 			(at 152.4 149.8599 0)
 			(effects
