File: boards/GIMIX 6809 CPU Plus/GIMIX 6809 CPU Plus/cpu.kicad_sch (KiCad schematic)
At the start: 25 parts, among them U26 74LS04, U27 74LS02, U33 74LS240, U34 74LS367, U47 MC6809, U48 74LS244, U51 74LS00, U52 74LS00, U53 74LS74, U54 74LS04

Commit message: CPU 6809 plus update
Parts:
- removed U34: 74LS367, Package_DIP:DIP-16_W7.62mm, symbol my_ics_new:74LS367_Split
- added U34: 74LS368, Package_DIP:DIP-16_W7.62mm, symbol my_ics_new:74LS368_Split
- R15, R20: value ? -> 10E
- R18, R8: value ? -> 1k
- R19, R21: value ? -> 22k
- R22: value ? -> 4k7
- RP3: value ? -> 10k
Connections:
- net BR/~{W}: now also U34.13
- net CE: now also U34.4
- net CQ: now also U34.6
- net CR/~{W}: now also U34.2
- net GND: now also U34.1
- net LW/~{R}: now also U34.14, U34.3
- net ~{BE}: now also U34.5
- net ~{BQ}: now also U34.7
- net ~{BVMA}: now also U34.11
- net at JA14.3 (Pin_3): now also U34.9
- net at U51.6: now also U34.10
- net at U51.8: now also U34.12
- net at U26.3, U52.6: now also U34.15
Other:
- note added: "74LS367 == DS8T97 74LS368 == DS8T98"
- note removed: "8T28 is the same as 74LS367."
