File: boards/GIMIX 6809 CPU Plus/GIMIX 6809 CPU Plus/io.kicad_sch (KiCad schematic)
At the start: 27 parts, among them U1 MM58167, U13 74LS123, U14 74LS74, U15 74LS00, U16 74LS32, U17 74LS136, U2 MC6840, U20 74LS12, U3 9511, Y1 32k768

Commit message: CPU 6809 plus update
Parts:
- R1: value ? -> 100E
- R17, R27, R6: value ? -> 4k7
Changed lines of the file:
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@@
 		(title "GIMIX 6809 CPU Plus")
 		(date "2026-07-02")
-		(rev "0.1")
+		(rev "0.2")
 		(company "100% Offner")
 		(comment 1 "v0.1: Initial")
+		(comment 2 "v0.2: ch. U34 -> 'LS368, ")
 	)
 	(text "check crystal!"
@@
 		(fields_autoplaced yes)
 		(property "Reference" "R1"
-			(at 260.35 24.13 90)
+			(at 260.35 22.86 90)
 			(effects
 				(font
@@
 			)
 		)
-		(property "Value" "?"
-			(at 260.35 26.67 90)
+		(property "Value" "100E"
+			(at 260.35 25.4 90)
 			(effects
 				(font
@@
 			)
 		)
-		(property "Value" "?"
+		(property "Value" "4k7"
 			(at 278.13 106.6799 0)
 			(effects
@@
 			)
 		)
-		(property "Value" "?"
+		(property "Value" "4k7"
 			(at 247.65 105.4099 0)
 			(effects
@@
 			)
 		)
-		(property "Value" "?"
+		(property "Value" "4k7"
 			(at 138.43 26.6699 0)
 			(effects
