File: boards/GIMIX 6809 CPU Plus/GIMIX 6809 CPU Plus/power.kicad_sch (KiCad schematic)
At the start: 71 parts, among them Q1 BC337, Q2 BC337, Q3 BC337, U10 74LS04, U13 74LS123, U14 74LS74, U15 74LS00, U16 74LS32, U17 74LS136, U18 74LS20, U19 74LS32, U20 74LS12, U25 74LS20, U26 74LS04, U27 74LS02, U28 LM7812_TO220, U29 LM7805_TO220, U30 LM7805_TO220, U31 LM7905_TO220, U32 74LS30, U33 74LS240, U34 74LS367, U35 74LS136, U46 74LS30, U48 74LS244, U51 74LS00, U52 74LS00, U53 74LS74, U54 74LS04

Commit message: CPU 6809 plus update
Parts:
- removed U34: 74LS367, Package_DIP:DIP-16_W7.62mm, symbol my_ics_new:74LS367_Split
- added U34: 74LS368, Package_DIP:DIP-16_W7.62mm, symbol my_ics_new:74LS368_Split
- D1: value ? -> 1N4001
- R11, R13, R4, R5: value ? -> 1k
- R14: value ? -> 10k
Connections:
- net +5A: now also U34.16 (VCC)
- net GND: now also U34.8 (GND)
Other:
- company: (none) -> 100% Offner
- title: (none) -> GIMIX 6809 CPU Plus
- moved on the sheet: C11, C12, C25, D4
