File: boards/GIMIX 6809 CPU Plus/GIMIX 6809 CPU Plus/rom.kicad_sch (KiCad schematic)
At the start: 22 parts, among them U19 74LS32, U20 74LS12, U33 74LS240, U4 27C32, U5 27C32, U6 27C32, U7 27C32, U8 2114, U9 2114

Commit message: CPU 6809 plus update
Parts:
- R2, R3: value ? -> 680E
Other:
- moved on the sheet: C29, C9, R3
Changed lines of the file:
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@@
 		(title "GIMIX 6809 CPU Plus")
 		(date "2026-07-02")
-		(rev "0.1")
+		(rev "0.2")
 		(company "100% Offner")
 		(comment 1 "v0.1: Initial")
+		(comment 2 "v0.2: ch. U34 -> 'LS368, ")
 	)
 	(junction
@@
 	)
 	(junction
-		(at 168.91 135.89)
+		(at 173.99 135.89)
 		(diameter 0)
 		(color 0 0 0 0)
@@
 	)
 	(junction
-		(at 161.29 135.89)
+		(at 163.83 135.89)
 		(diameter 0)
 		(color 0 0 0 0)
@@
 	)
 	(junction
-		(at 168.91 144.78)
+		(at 173.99 144.78)
 		(diameter 0)
 		(color 0 0 0 0)
@@
 	(wire
 		(pts
-			(xy 161.29 135.89) (xy 161.29 137.16)
+			(xy 163.83 135.89) (xy 163.83 137.16)
 		)
 		(stroke
@@
 	(wire
 		(pts
-			(xy 168.91 144.78) (xy 168.91 143.51)
+			(xy 173.99 144.78) (xy 173.99 143.51)
 		)
 		(stroke
@@
 	(wire
 		(pts
-			(xy 176.53 135.89) (xy 168.91 135.89)
+			(xy 181.61 135.89) (xy 173.99 135.89)
 		)
 		(stroke
@@
 	(wire
 		(pts
-			(xy 161.29 142.24) (xy 161.29 151.13)
+			(xy 163.83 142.24) (xy 163.83 151.13)
 		)
 		(stroke
@@
 	(wire
 		(pts
-			(xy 168.91 135.89) (xy 168.91 138.43)
+			(xy 173.99 135.89) (xy 173.99 138.43)
 		)
 		(stroke
@@
 	(wire
 		(pts
-			(xy 161.29 135.89) (xy 168.91 135.89)
+			(xy 163.83 135.89) (xy 173.99 135.89)
 		)
 		(stroke
@@
 	(wire
 		(pts
-			(xy 154.94 135.89) (xy 161.29 135.89)
+			(xy 154.94 135.89) (xy 163.83 135.89)
 		)
 		(stroke
@@
 	(wire
 		(pts
-			(xy 176.53 138.43) (xy 176.53 135.89)
+			(xy 181.61 138.43) (xy 181.61 135.89)
 		)
 		(stroke
@@
 	(wire
 		(pts
-			(xy 176.53 144.78) (xy 168.91 144.78)
+			(xy 181.61 144.78) (xy 173.99 144.78)
 		)
 		(stroke
@@
 	(wire
 		(pts
-			(xy 168.91 146.05) (xy 168.91 144.78)
+			(xy 173.99 146.05) (xy 173.99 144.78)
 		)
 		(stroke
@@
 	(wire
 		(pts
-			(xy 176.53 143.51) (xy 176.53 144.78)
+			(xy 181.61 143.51) (xy 181.61 144.78)
 		)
 		(stroke
@@
 	)
 	(label "~{WRAM}"
-		(at 161.29 151.13 90)
+		(at 163.83 151.13 90)
 		(effects
 			(font
@@
 	(symbol
 		(lib_id "Device:C_Small")
-		(at 168.91 140.97 0)
+		(at 173.99 140.97 0)
 		(unit 1)
 		(exclude_from_sim no)
@@
 		(fields_autoplaced yes)
 		(property "Reference" "C9"
-			(at 171.45 139.7062 0)
+			(at 176.53 139.7062 0)
 			(effects
 				(font
@@
 		)
 		(property "Value" "?"
-			(at 171.45 142.2462 0)
+			(at 176.53 142.2462 0)
 			(effects
 				(font
@@
 		)
 		(property "Footprint" "Capacitor_THT:C_Disc_D3.8mm_W2.6mm_P2.50mm"
-			(at 168.91 140.97 0)
+			(at 173.99 140.97 0)
 			(effects
 				(font
@@
 		)
 		(property "Datasheet" "~"
-			(at 168.91 140.97 0)
+			(at 173.99 140.97 0)
 			(effects
 				(font
@@
 		)
 		(property "Description" "Unpolarized capacitor, small symbol"
-			(at 168.91 140.97 0)
+			(at 173.99 140.97 0)
 			(effects
 				(font
@@
 	(symbol
 		(lib_id "Device:R_Small")
-		(at 161.29 139.7 0)
+		(at 163.83 139.7 0)
 		(unit 1)
 		(exclude_from_sim no)
@@
 		(fields_autoplaced yes)
 		(property "Reference" "R3"
-			(at 163.83 138.4299 0)
+			(at 166.37 138.4299 0)
 			(effects
 				(font
@@
 			)
 		)
-		(property "Value" "?"
-			(at 163.83 140.9699 0)
+		(property "Value" "680E"
+			(at 166.37 140.9699 0)
 			(effects
 				(font
@@
 		)
 		(property "Footprint" "Resistor_THT:R_Axial_DIN0207_L6.3mm_D2.5mm_P10.16mm_Horizontal"
-			(at 161.29 139.7 0)
+			(at 163.83 139.7 0)
 			(effects
 				(font
@@
 		)
 		(property "Datasheet" "~"
-			(at 161.29 139.7 0)
+			(at 163.83 139.7 0)
 			(effects
 				(font
@@
 		)
 		(property "Description" "Resistor, small symbol"
-			(at 161.29 139.7 0)
+			(at 163.83 139.7 0)
 			(effects
 				(font
@@
 	(symbol
 		(lib_id "power:GND")
-		(at 168.91 146.05 0)
+		(at 173.99 146.05 0)
 		(unit 1)
 		(exclude_from_sim no)
@@
 		(fields_autoplaced yes)
 		(property "Reference" "#PWR0119"
-			(at 168.91 152.4 0)
+			(at 173.99 152.4 0)
 			(effects
 				(font
@@
 		)
 		(property "Value" "GND"
-			(at 168.91 151.13 0)
+			(at 173.99 151.13 0)
 			(effects
 				(font
@@
 		)
 		(property "Footprint" ""
-			(at 168.91 146.05 0)
+			(at 173.99 146.05 0)
 			(effects
 				(font
@@
 		)
 		(property "Datasheet" ""
-			(at 168.91 146.05 0)
+			(at 173.99 146.05 0)
 			(effects
 				(font
@@
 		)
 		(property "Description" "Power symbol creates a global label with name \"GND\" , ground"
-			(at 168.91 146.05 0)
+			(at 173.99 146.05 0)
 			(effects
 				(font
@@
 			)
 		)
-		(property "Value" "?"
+		(property "Value" "680E"
 			(at 157.48 140.9699 0)
 			(effects
@@
 	(symbol
 		(lib_id "Device:C_Small")
-		(at 176.53 140.97 0)
+		(at 181.61 140.97 0)
 		(unit 1)
 		(exclude_from_sim no)
@@
 		(fields_autoplaced yes)
 		(property "Reference" "C29"
-			(at 179.07 139.7062 0)
+			(at 184.15 139.7062 0)
 			(effects
 				(font
@@
 		)
 		(property "Value" "?"
-			(at 179.07 142.2462 0)
+			(at 184.15 142.2462 0)
 			(effects
 				(font
@@
 		)
 		(property "Footprint" "Capacitor_THT:C_Disc_D3.8mm_W2.6mm_P2.50mm"
-			(at 176.53 140.97 0)
+			(at 181.61 140.97 0)
 			(effects
 				(font
@@
 		)
 		(property "Datasheet" "~"
-			(at 176.53 140.97 0)
+			(at 181.61 140.97 0)
 			(effects
 				(font
@@
 		)
 		(property "Description" "Unpolarized capacitor, small symbol"
-			(at 176.53 140.97 0)
+			(at 181.61 140.97 0)
 			(effects
 				(font
