File: boards/GIMIX 256k SRAM/GIMIX 256k SRAM/GIMIX 256k SRAM.kicad_sch (KiCad schematic)
At the start: 29 parts, among them P1 SS-50 Bus, U33 74LS138, U34 74LS138, U35 74LS138, U36 74F244, U37 74LS138, U39 PAL16L8, U40 74F244, U41 74F244, U42 74LS640, U49 74LS641

Commit message: some info added
Other:
- note added: "-> -> <- -> -> -> -> ->"
Changed lines of the file:
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@@
 		(title "GIMIX 256k SRAM")
 		(date "2026-07-01")
-		(rev "0.1")
+		(rev "0.11")
 		(company "100% Offner")
 		(comment 1 "v0.1: Initial")
+		(comment 2 "v0.11: only direction to the PAL added.")
 	)
 	(text "JP1-5 are Solder Jumpers and\nare only for 62256 RAM Chips\nused."
@@
 		)
 	)
+	(text "->\n->\n<-\n->\n->\n->\n->\n->\n"
+		(exclude_from_sim no)
+		(at 273.558 192.024 0)
+		(effects
+			(font
+				(size 1.6002 1.6002)
+			)
+		)
+	)
