File: boards/GIMIX 256k SRAM/GIMIX 256k SRAM/power.kicad_sch (KiCad schematic)
At the start: 48 parts, among them Q1 BC337, Q2 BC337, U46 LM7805_TO220, U47 LM7805_TO220, U48 LM7805_TO220

Commit message: 256k RAM production version added
Parts:
- BT1: footprint (none) -> Connector_PinHeader_2.54mm:PinHeader_1x02_P2.54mm_Vertical
Changed lines of the file:
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@@
 			)
 		)
-		(property "Footprint" ""
+		(property "Footprint" "Connector_PinHeader_2.54mm:PinHeader_1x02_P2.54mm_Vertical"
 			(at 68.58 48.006 90)
 			(effects
