File: boards/GIMIX Serial intelligent/GIMIX intelligent 3 port Serial/GIMIX intelligent 3 port Serial.kicad_sch (KiCad schematic)
At the start: 45 parts, among them J1 SS30 Bus, SW1 SW_DIP_x08, SW2 SW_DIP_x08, U1 Z8038, U10 2764, U11 6116, U12 2764, U13 6551, U14 6551, U15 6551, U2 PAL16L8, U3 MC68B09, U4 74LS221, U5 7404, U6 74LS138, U7 74LS540, U8 74LS540, U9 6116, Y1 8M?, Y2 8M?

Commit message: some info added
Connections:
- net ~{ZRD}: now reaches U1.3 (CA), U2.16 (IO4)
- net ~{ZWR}: now reaches U1.4 (DA), U2.15 (IO5)
- net ~{ZCE}: now reaches U1.5 (EA), U2.14 (IO6)
- net ~{ZINTACK}: now reaches U1.7 (GA), U2.13 (IO7)
Other:
- note added: "-> -> -> -> -> -> -> ->"
- note added: "Z8038 Mode: 8-11 (Non-Z-BUS)"
