File: boards/GIMIX DMA Floppy/GIMIX DMA Floppy_v1.0/GIMIX DMA Floppy.kicad_pcb (KiCad board)
At the start: 2 copper layers, 248.9 x 139.7 mm, 136 parts, among them J1 Floppy 5.25", J2 Floppy 8", P1 SS-50 Bus, Q1 LM7805_TO220, Q2 LM7805_TO220, SW1 SW_DIP_x10, SW2 SW_DIP_x10, U1 74LS244, U10 74LS393, U11 7404, U12 74LS74, U14 74LS08, U19 WD2797, U2 7438, U20 4538, U22 74LS123, U23 7406, U24 74LS74, U25 74LS74, U26 74LS367, U27 74LS138, U28 74LS273, U29 74LS174, U3 7438, U30 74LS161, U31 74LS161, U32 74LS161, U33 74LS161, U34 74LS240, U35 74LS240, U36 74F04, U37 7420, U38 74LS367, U39 74LS32, U4 7406, U40 74LS136, U41 74LS136, U42 74LS136, U43 74LS136, U44 74LS136, U45 74LS244, U46 74LS244, U47 74LS533, U48 74LS244, U5 7406, U52 74LS132, U54 74LS161, U55 7406, U59 74LS74, U6 74LS08, U7 74LS08, U8 74LS157, U9 74LS221, Y1 ?

Commit message: DMA Floppy silkscreen and gerbers added
Parts:
- C18: value C_Small -> 0
- R10: value ? -> 9k1
- R11: value ? -> 330E
- R12, R13: value R_Small -> 680E
- R16, R36, R40, R41, R44: value ? -> 680E
- R2: value ? -> 1M5
- R3: value ? -> 15k
- R35: value ? -> 0E
- R37, R38, R64, R8: value ? -> 1k
- R39, R46: value ? -> 10k
- R42: value ? -> 30k
- R43: value ? -> 4k7
- R6: value ? -> 100k
- R65, R66: value ? -> 18k
- R7: value ? -> 2k2
- R9: value ? -> 13k
Connections:
- U23 pad 1: unconnected-(U23-Pad1) -> GND
- U23 pad 13: unconnected-(U23-Pad13) -> GND
- U23 pad 5: unconnected-(U23-Pad5) -> GND
- U36 pad 11: unconnected-(U36-Pad11) -> GND
- U55 pad 9: unconnected-(U55-Pad9) -> GND
Routing:
- net GND: track 1445.0 -> 1486.3 mm, vias 12 -> 33
- net /~{RE}: track 344.5 -> 348.0 mm
- net Net-(U59A-C): track 224.5 -> 226.2 mm
- net /Floppy Controller/U1-12: track 249.7 -> 251.3 mm
- net /Floppy Controller/HDLD: track 315.5 -> 314.1 mm
- net Net-(U22A-A): track 193.7 -> 194.7 mm
- net Net-(U25A-~{Q}): track 264.7 -> 265.4 mm
Other:
- board text added: "Reproduction 100% Offner 2026 v1.0"
- board text removed: "Reproduction 100% Offner 2026"
