File: boards/GIMIX DMA Floppy/GIMIX DMA Floppy_v1.0/GIMIX DMA Floppy.kicad_sch (KiCad schematic)
At the start: 24 parts, among them P1 SS-50 Bus, U10 74LS393, U11 7404, U14 74LS08, U23 7406, U24 74LS74, U25 74LS74, U27 74LS138, U28 74LS273, U29 74LS174, U34 74LS240, U35 74LS240, U36 74F04, U37 7420, U38 74LS367, U39 74LS32, U41 74LS136, U47 74LS533, U48 74LS244, U6 74LS08, U7 74LS08

Commit message: DMA Floppy silkscreen and gerbers added
Parts:
- R40: value ? -> 680E
Changed lines of the file:
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@@
 			)
 		)
-		(property "Value" "?"
+		(property "Value" "680E"
 			(at 214.63 135.8899 0)
 			(effects
