File: boards/GIMIX DMA Floppy/GIMIX DMA Floppy_v1.0/dma.kicad_sch (KiCad schematic)
At the start: 10 parts, among them U30 74LS161, U31 74LS161, U32 74LS161, U33 74LS161, U38 74LS367, U45 74LS244, U46 74LS244, U54 74LS161

Commit message: DMA Floppy silkscreen and gerbers added
Parts:
- R43: value ? -> 4k7
Changed lines of the file:
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@@
 			)
 		)
-		(property "Value" "?"
+		(property "Value" "4k7"
 			(at 110.49 217.1699 0)
 			(effects
