File: boards/GIMIX DMA Floppy/GIMIX DMA Floppy_v1.0/floppy.kicad_sch (KiCad schematic)
At the start: 73 parts, among them J1 Floppy 5.25", J2 Floppy 8", U1 74LS244, U11 7404, U12 74LS74, U14 74LS08, U19 WD2797, U2 7438, U20 4538, U22 74LS123, U23 7406, U25 74LS74, U26 74LS367, U3 7438, U4 7406, U5 7406, U52 74LS132, U55 7406, U59 74LS74, U6 74LS08, U7 74LS08, U8 74LS157, U9 74LS221, Y1 ?

Commit message: DMA Floppy silkscreen and gerbers added
Parts:
- R10: value ? -> 9k1
- R11: value ? -> 330E
- R12, R13: value R_Small -> 680E
- R2: value ? -> 1M5
- R3: value ? -> 15k
- R37, R38, R64, R8: value ? -> 1k
- R39, R46: value ? -> 10k
- R42: value ? -> 30k
- R6: value ? -> 100k
- R65, R66: value ? -> 18k
- R7: value ? -> 2k2
- R9: value ? -> 13k
Changed lines of the file:
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@@
 			)
 		)
-		(property "Value" "?"
+		(property "Value" "10k"
 			(at 204.47 264.1599 0)
 			(effects
@@
 			)
 		)
-		(property "Value" "?"
+		(property "Value" "30k"
 			(at 83.82 95.2499 0)
 			(effects
@@
 			)
 		)
-		(property "Value" "?"
+		(property "Value" "2k2"
 			(at 327.66 223.5199 0)
 			(effects
@@
 			)
 		)
-		(property "Value" "?"
+		(property "Value" "330E"
 			(at 254 22.8599 0)
 			(effects
@@
 			)
 		)
-		(property "Value" "?"
+		(property "Value" "18k"
 			(at 73.66 193.0399 0)
 			(effects
@@
 			)
 		)
-		(property "Value" "R_Small"
+		(property "Value" "680E"
 			(at 25.4 16.51 90)
 			(effects
@@
 			)
 		)
-		(property "Value" "?"
+		(property "Value" "18k"
 			(at 66.04 252.7299 0)
 			(effects
@@
 			)
 		)
-		(property "Value" "?"
+		(property "Value" "1M5"
 			(at 372.11 140.9699 0)
 			(effects
@@
 			)
 		)
-		(property "Value" "?"
+		(property "Value" "1k"
 			(at 43.18 190.4999 0)
 			(effects
@@
 			)
 		)
-		(property "Value" "?"
+		(property "Value" "1k"
 			(at 344.17 160.0199 0)
 			(effects
@@
 			)
 		)
-		(property "Value" "?"
+		(property "Value" "1k"
 			(at 85.09 186.6899 0)
 			(effects
@@
 			)
 		)
-		(property "Value" "?"
+		(property "Value" "10k"
 			(at 74.93 95.2499 0)
 			(effects
@@
 			)
 		)
-		(property "Value" "?"
+		(property "Value" "100k"
 			(at 100.33 212.0899 0)
 			(effects
@@
 			)
 		)
-		(property "Value" "?"
+		(property "Value" "13k"
 			(at 279.4 44.4499 0)
 			(effects
@@
 			)
 		)
-		(property "Value" "?"
+		(property "Value" "9k1"
 			(at 278.13 81.2799 0)
 			(effects
@@
 			)
 		)
-		(property "Value" "?"
+		(property "Value" "15k"
 			(at 372.11 182.8799 0)
 			(effects
@@
 			)
 		)
-		(property "Value" "?"
+		(property "Value" "1k"
 			(at 140.97 109.2199 0)
 			(effects
@@
 			)
 		)
-		(property "Value" "R_Small"
+		(property "Value" "680E"
 			(at 43.18 16.51 90)
 			(effects
