File: boards/GIMIX DMA Floppy/GIMIX DMA Floppy_v1.0/floppy.kicad_sch (KiCad schematic)
At the start: 76 parts, among them J1 Floppy 5.25", J2 Floppy 8", U1 74LS244, U11 7404, U12 74LS74, U14 74LS08, U19 WD2797, U2 7438, U20 4538, U22 74LS123, U23 7406, U25 74LS74, U26 74LS367, U3 7438, U4 7406, U5 7406, U52 74LS132, U55 7406, U59 74LS74, U6 74LS08, U7 74LS08, U8 74LS157, U9 74LS221, Y1 ?

Commit message: boms added
Parts:
- Y1: value ? -> 4M
Changed lines of the file:
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@@
 			)
 		)
-		(property "Value" "?"
+		(property "Value" "4M"
 			(at 33.02 35.56 0)
 			(effects
