File: boards/GIMIX DMA Floppy/GIMIX DMA Floppy_v1.0/power.kicad_sch (KiCad schematic)
At the start: 54 parts, among them Q1 LM7805_TO220, Q2 LM7805_TO220, U10 74LS393, U11 7404, U12 74LS74, U14 74LS08, U2 7438, U20 4538, U22 74LS123, U23 7406, U24 74LS74, U25 74LS74, U3 7438, U36 74F04, U37 7420, U38 74LS367, U39 74LS32, U4 7406, U40 74LS136, U41 74LS136, U42 74LS136, U43 74LS136, U44 74LS136, U45 74LS244, U46 74LS244, U5 7406, U52 74LS132, U55 7406, U59 74LS74, U6 74LS08, U7 74LS08, U9 74LS221

Commit message: DMA Floppy silkscreen and gerbers added
Parts:
- R16, R41: value ? -> 680E
Connections:
- net GND: now also U23.1, U23.13, U23.5, U36.11, U55.9
- no-connect marks 0 -> 5
