File: boards/GIMIX DMA Floppy/GIMIX DMA Floppy/GIMIX DMA Floppy.kicad_pcb (KiCad board)
At the start: 2 copper layers, 248.9 x 139.7 mm, 138 parts, among them J1 Floppy 5.25", J2 Floppy 8", P1 SS-50 Bus, Q1 LM7805_TO220, Q2 LM7805_TO220, SW1 SW_DIP_x10, SW2 SW_DIP_x10, U1 74LS244, U10 74LS393, U11 7404, U12 74LS74, U14 74LS08, U19 WD2797, U2 7438, U20 4538, U22 74LS123, U23 7406, U24 74LS74, U25 74LS74, U26 74LS367, U27 74LS138, U28 74LS273, U29 74LS174, U3 7438, U30 74LS161, U31 74LS161, U32 74LS161, U33 74LS161, U34 74LS240, U35 74LS240, U36 74F04, U37 7420, U38 74LS367, U39 74LS32, U4 7406, U40 74LS136, U41 74LS136, U42 74LS136, U43 74LS136, U44 74LS136, U45 74LS244, U46 74LS244, U47 74LS533, U48 74LS244, U5 7406, U52 74LS132, U54 74LS161, U55 7406, U59 74LS74, U6 74LS08, U7 74LS08, U8 74LS157, U9 74LS221, Y1 ?

Commit message: DMA Floppy update, silkscreen and gerbers added
Parts:
- removed Cx1, Cx2: ?, Capacitor_SMD:C_1206_3216Metric_Pad1.33x1.80mm_HandSolder
- C31: footprint my_own:Capacitor_Trim -> Potentiometer_THT:Potentiometer_Piher_PT-10-V05_Vertical
- JA1: value RDY Option -> RDY Select
- JA10: value Software Writeprotect Option -> WP Select
- JA11: value Reserved -> WP Select
- JA12: value BA/BS Select -> BS Select
- JA13: value DMA Option -> HALT/BREQ Select
- JA14: value Slow Memory Option -> ? Select
- JA16: value 8" MOT Select -> MOT Select
- JA17: value 8" Headload Delay -> ? Select
- JA2: value Headload Option -> Headload Select
- JA20: value DMA Extended Address Counter -> Jumper_3_Bridged12
- JA3: value DRV3 Option -> DRV3 Select
- JA6: value 5.25" and 8" Precomp Option -> Conn_02x05_Odd_Even
- JA7: value Motor On Delay Option -> ? Select
- JA8: value Head Load Option -> ? Select
- RP2, RP3: value 10k -> ?
- moved C31 9.97 mm to (241.0, 56.1), turned to -90 degrees
- moved C44 5.43 mm to (149.2, 40.8), turned to 0 degrees
- moved C8 2.51 mm to (146.1, 59.4), turned to 90 degrees
- moved R38 1.52 mm to (237.2, 51.1)
- moved C49 1.30 mm to (138.2, 120.4)
- moved R64 1.14 mm to (228.3, 67.1)
- moved D1 1.09 mm to (225.0, 67.1)
- moved C20 1.02 mm to (232.7, 56.9)
- moved C32 0.63 mm to (240.0, 48.3)
- moved C45 0.57 mm to (175.3, 30.2)
- moved C50 0.51 mm to (207.0, 152.9)
- moved R8 0.51 mm to (124.2, 83.6)
- moved C6 0.25 mm to (79.5, 96.0)
- moved JA16 0.25 mm to (80.3, 71.1)
- moved J1 0.13 mm to (71.6, 32.9)
Connections:
- C31 pad 1: Net-(C31-Pad1) -> GND
Routing:
- net GND: track 1950.4 -> 1486.3 mm, vias 67 -> 33
- net +5V: track 620.8 -> 471.4 mm, vias 9 -> 3
- net /~{RST}: track 588.7 -> 660.3 mm, vias 12 -> 8
- net /~{LDL}: track 198.7 -> 266.2 mm, vias 1 -> 4
- net /DRQ#: track 212.4 -> 269.7 mm
- net +5C: track 818.3 -> 872.5 mm, vias 17 -> 7
- net /U34-13: track 269.5 -> 314.0 mm
- net /Floppy Controller/~{5}/8: track 269.2 -> 227.2 mm, vias 6 -> 5
- net Net-(U59A-C): track 187.8 -> 226.2 mm, vias 2 -> 5
- net Net-(U25A-~{Q}): track 231.7 -> 265.4 mm, vias 0 -> 2
- net /ID2: track 251.9 -> 284.1 mm, vias 3 -> 4
- net /~{LDH}: track 90.9 -> 122.7 mm, vias 2 -> 4
- net /Floppy Controller/ENP: track 184.0 -> 214.2 mm
- net Net-(R44-Pad2): track 177.8 -> 207.8 mm
- net /A19: track 113.4 -> 142.5 mm
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Other:
- board text added: "Reproduction 100% Offner 2026 NOT for Production!"
- board text removed: "Adjustment: set TP5 to GND AFTER Reset. adj. C31 for 500kHz on Pin 16 (TP3), RPW for 250ns on Pin 29 (TP2) and WPW for 125ns on Pin 31 (T4P)."
- board text removed: "GND"
- board text removed: "Reproduction 100% Offner 2026 v1.0"
- board text removed: "TP1"
- board text removed: "TP2"
- board text removed: "TP3"
- board text removed: "TP4"
- board text removed: "TP5"
