File: boards/GIMIX DMA Floppy/GIMIX DMA Floppy/GIMIX DMA Floppy.kicad_pcb (KiCad board)
At the start: 2 copper layers, 248.9 x 139.7 mm, 136 parts, among them J1 Floppy 5.25", J2 Floppy 8", P1 SS-50 Bus, Q1 LM7805_TO220, Q2 LM7805_TO220, SW1 SW_DIP_x10, SW2 SW_DIP_x10, U1 74LS244, U10 74LS393, U11 7404, U12 74LS74, U14 74LS08, U19 WD2797, U2 7438, U20 4538, U22 74LS123, U23 7406, U24 74LS74, U25 74LS74, U26 74LS367, U27 74LS138, U28 74LS273, U29 74LS174, U3 7438, U30 74LS161, U31 74LS161, U32 74LS161, U33 74LS161, U34 74LS240, U35 74LS240, U36 74F04, U37 7420, U38 74LS367, U39 74LS32, U4 7406, U40 74LS136, U41 74LS136, U42 74LS136, U43 74LS136, U44 74LS136, U45 74LS244, U46 74LS244, U47 74LS533, U48 74LS244, U5 7406, U52 74LS132, U54 74LS161, U55 7406, U59 74LS74, U6 74LS08, U7 74LS08, U8 74LS157, U9 74LS221, Y1 ?

Commit message: original DMA Floppy update
Routing:
- net GND: track 1486.3 -> 1530.8 mm, vias 33 -> 17
- net /~{LDL}: track 266.2 -> 303.1 mm
- net /IRQ: track 157.3 -> 154.1 mm
- net /Floppy Controller/~{5}/8: track 227.2 -> 229.5 mm
- net Net-(U12A-D): track 13.0 -> 11.8 mm
- net /Floppy Controller/DRQ: track 210.7 -> 209.5 mm
- net TP1: track 59.3 -> 58.2 mm
- net /A7_out: track 203.2 -> 202.6 mm
- net /Floppy Controller/~{8}/5: track 158.7 -> 158.1 mm
- net /Floppy Controller/RDY: track 131.4 -> 130.8 mm
- removed copper zone on B.Cu, net GND
- removed copper zone on F.Cu, net GND
