File: boards/GIMIX DMA Floppy/GIMIX DMA Floppy/floppy.kicad_sch (KiCad schematic)
At the start: 76 parts, among them J1 Floppy 5.25", J2 Floppy 8", U1 74LS244, U11 7404, U12 74LS74, U14 74LS08, U19 WD2797, U2 7438, U20 4538, U22 74LS123, U23 7406, U25 74LS74, U26 74LS367, U3 7438, U4 7406, U5 7406, U52 74LS132, U55 7406, U59 74LS74, U6 74LS08, U7 74LS08, U8 74LS157, U9 74LS221, Y1 ?

Commit message: DMA Floppy update, silkscreen and gerbers added
Parts:
- removed Cx1, Cx2: ?, Capacitor_SMD:C_1206_3216Metric_Pad1.33x1.80mm_HandSolder, symbol Device:C_Small
- removed JA18: TESTPOINTS, Connector_PinHeader_2.54mm:PinHeader_1x06_P2.54mm_Vertical, symbol Connector_Generic:Conn_01x06
- C31: footprint my_own:Capacitor_Trim -> Potentiometer_THT:Potentiometer_Piher_PT-10-V05_Vertical
- JA1: value RDY Option -> RDY Select
- JA10: value Software Writeprotect Option -> WP Select
- JA11: value Reserved -> WP Select
- JA14: value Slow Memory Option -> ? Select
- JA16: value 8" MOT Select -> MOT Select
- JA17: value 8" Headload Delay -> ? Select
- JA2: value Headload Option -> Headload Select
- JA3: value DRV3 Option -> DRV3 Select
- JA6: value 5.25" and 8" Precomp Option -> Conn_02x05_Odd_Even
- JA7: value Motor On Delay Option -> ? Select
- JA8: value Head Load Option -> ? Select
Connections:
- net GND: now also C31.1
Other:
- note removed: "Adjustment: set TP5 to GND AFTER Reset. adj. C31 for 500kHz on Pin 16 (TP3), RPW for 250ns on Pin 29 (TP2) and WPW for 125ns on Pin 31 (T4P)."
- note removed: "JA10: 1-2"
- note removed: "JA11: 1-2"
- note removed: "JA14: 1-2"
- note removed: "JA15: 3-4"
- note removed: "JA16: 2-3"
- note removed: "JA17: 1-2"
- note removed: "JA1: 3-4"
- note removed: "JA2: open"
- note removed: "JA3: 2-3"
- note removed: "JA4: 2-3"
- note removed: "JA5: 1-2"
- note removed: "JA6: 5-6 and 7-8"
- note removed: "JA7: 1-2"
- note removed: "JA8: 1-2"
- moved on the sheet: C8, JA17, JA6, JA7, JA8, R10, U11B, U7C, U8, U9A
