File: boards/GIMIX BaudRateGenerator/GIMIX BaudRateGenerator/GIMIX BaudRateGenerator.kicad_pcb (KiCad board)
At the start: 2 copper layers, 58.4 x 83.8 mm, 19 parts, among them J1 Mainboard, J2 Conn_01x05, J4 A, J5 B, J6 C, J7 D, J8 E, J9 Conn_02x05_Odd_Even, U1 MC14411, U2 4512, U3 4069, U4 74LS244, Y1 1M8324

Commit message: DMA SASI update
Parts:
- R1: value ? -> 10M
- renumbered J2 to CA1
Changed lines of the file:
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@@
 			)
 		)
-		(property "Value" "?"
+		(property "Value" "10M"
 			(at 5.08 2.37 0)
 			(layer "F.Fab")
@@
 		(descr "Through hole straight pin header, 1x05, 2.54mm pitch, single row")
 		(tags "Through hole pin header THT 1x05 2.54mm single row")
-		(property "Reference" "J2"
+		(property "Reference" "CA1"
 			(at 0 -2.38 0)
 			(layer "F.SilkS")
