File: boards/GIMIX BaudRateGenerator/GIMIX BaudRateGenerator/GIMIX BaudRateGenerator.kicad_sch (KiCad schematic)
At the start: 19 parts, among them J1 Mainboard, J2 Conn_01x05, J3 Range, J4 A, J5 B, J6 C, J7 D, J8 E, J9 Conn_02x05_Odd_Even, U1 MC14411, U2 4512, U3 4069, U4 74LS244, Y1 1M8324

Commit message: Baudrate Gen. silkscreen and gerbers added
Parts:
- renumbered J2 to CA1, J3 to JA1
Changed lines of the file:
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@@
 		(dnp no)
 		(fields_autoplaced yes)
-		(property "Reference" "J3"
+		(property "Reference" "JA1"
 			(at 15.24 21.59 0)
 			(effects
@@
 			(project "GIMIX BaudRateGenerator"
 				(path "/70168188-e4e4-4916-9756-ee4bf3545c70"
-					(reference "J3")
+					(reference "JA1")
 					(unit 1)
 				)
@@
 		(on_board yes)
 		(dnp no)
-		(property "Reference" "J2"
-			(at 24.892 95.758 0)
+		(property "Reference" "CA1"
+			(at 21.59 95.758 0)
 			(effects
 				(font
@@
 			(project "GIMIX BaudRateGenerator"
 				(path "/70168188-e4e4-4916-9756-ee4bf3545c70"
-					(reference "J2")
+					(reference "CA1")
 					(unit 1)
 				)

Commit message: DMA SASI update
Parts:
- R1: value ? -> 10M
Changed lines of the file:
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@@
 		(title "GIMIX Baud Rate Generator Board")
 		(date "2026-06-25")
-		(rev "0.1")
+		(rev "0.2")
 		(company "100% Offner")
 		(comment 1 "v0.1: Initial")
+		(comment 2 "v0.2: R1 added")
 	)
 	(junction
@@
 			)
 		)
-		(property "Value" "?"
+		(property "Value" "10M"
 			(at 21.59 76.2 90)
 			(effects
