File: boards/GIMIX DMA SASI/GIMIX DMA SASI_production/GIMIX DMA SASI.kicad_pcb (KiCad board)
At the start: 2 copper layers, 249.9 x 140.7 mm, 83 parts, among them J1 Power, J19 Conn_02x03_Odd_Even, J2 SASI, J3 Conn_01x20, P1 SS-50 Bus, SW1 SW_DIP_x10, SW2 SW_DIP_x10, U1 7438, U10 74LS32, U11 74LS240, U12 74LS138, U13 74LS367, U14 74LS161, U15 7474, U16 74LS08, U17 7474, U18 74LS10, U19 74LS240, U2 74LS08, U20 74LS136, U21 74LS136, U22 74LS136, U23 74LS136, U24 74LS136, U25 74LS161, U26 74LS161, U27 74LS161, U28 74LS161, U29 74LS273, U3 74LS74, U30 74LS273, U31 74LS240, U32 74LS244, U33 LM7805_TO220, U34 LM7805_TO220, U35 74LS244, U36 74LS244, U37 74LS240, U38 LM7805_TO220, U4 74LS74, U5 74LS20, U6 7438, U7 7438, U8 7438, U9 7438

Commit message: DMA SASI update
Parts:
- added TP1: SASIR, Connector_PinHeader_2.54mm:PinHeader_1x01_P2.54mm_Vertical, B.Cu at (242.7, 82.3)
- added TP2: SASIW, Connector_PinHeader_2.54mm:PinHeader_1x01_P2.54mm_Vertical, B.Cu at (232.5, 75.4)
- added TP3: WE, Connector_PinHeader_2.54mm:PinHeader_1x01_P2.54mm_Vertical, B.Cu at (213.7, 71.6)
- added TP4: RE, Connector_PinHeader_2.54mm:PinHeader_1x01_P2.54mm_Vertical, B.Cu at (269.6, 80.9)
- added TP5: OutputBuffer On, Connector_PinHeader_2.54mm:PinHeader_1x01_P2.54mm_Vertical, B.Cu at (236.3, 16.4)
- added TP6: StatusBuffer On, Connector_PinHeader_2.54mm:PinHeader_1x01_P2.54mm_Vertical, B.Cu at (245.7, 36.2)
- J3: value Conn_01x20 -> Debug
- R1: value ? -> 10E
- R2, R3, R5: value ? -> 680E
- R4: value ? -> 4k7
- R6: value ? -> 470E
- R7: value ? -> 1k
- RP1, RP2: value ? -> 10k
Routing:
- net /~{SASIR}: track 141.9 -> 147.2 mm
- net /~{SASIW}: track 174.2 -> 178.8 mm
- net /SASI Interface/~{SD5}: track 129.8 -> 133.4 mm
- net /SASI Interface/~{SD6}: track 160.7 -> 157.3 mm
- net /~{RE}: track 218.8 -> 221.9 mm
- net /SASI Interface/SAD2: track 86.7 -> 88.3 mm
- net /SASI Interface/~{SD7}: track 182.2 -> 180.8 mm
- net Net-(U15A-Q): track 149.1 -> 148.4 mm, vias 4 -> 3
- net /~{WE}: track 145.9 -> 146.1 mm, vias 5 -> 4
Other:
- board text added: "Output Buffer On"
- board text added: "Remake by 100% Offner 2026 v1.1"
- board text added: "Status Buffer On"
- board text added: "~{RE}"
- board text added: "~{SASIR}"
- board text added: "~{SASIW}"
- board text added: "~{WE}"
- board text removed: "Remake by 100% Offner 2026 v1.0"
