File: boards/GIMIX DMA SASI/GIMIX DMA SASI_production/GIMIX DMA SASI.kicad_sch (KiCad schematic)
At the start: 14 parts, among them J19 Conn_02x03_Odd_Even, P1 SS-50 Bus, U1 7438, U11 74LS240, U12 74LS138, U13 74LS367, U2 74LS08, U20 74LS136, U3 74LS74, U37 74LS240, U4 74LS74, U5 74LS20

Commit message: DMA SASI update
Parts:
- R3: value ? -> 680E
- R4: value ? -> 4k7
Changed lines of the file:
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@@
 		(title "GIMIX DMA SASI Controller")
 		(date "2026-06-15")
-		(rev "0.4")
+		(rev "0.5")
 		(company "100% Offner")
-		(comment 1 "v0.1: Initial")
-		(comment 2 "v0.2: cleanup for production, gerbers exported")
-		(comment 3 "v0.3: third regulator added.")
-		(comment 4 "v0.4: add BlueSCSI v2 Mounting Holes, rotate 50p conn., add Logic Anlyzer Pins")
+		(comment 1 "v0.4: add BlueSCSI v2 Mounting Holes, rotate 50p conn., add Logic Anlyzer Pins")
+		(comment 2 "v0.5: Resistor Values and more Testpoints added")
 	)
 	(text "on GIMIX\nBE and BQ\nare inverted.\nCheck with CMS!"
@@
 			)
 		)
-		(property "Value" "?"
+		(property "Value" "4k7"
 			(at 43.18 219.7099 0)
 			(effects
@@
 			)
 		)
-		(property "Value" "?"
+		(property "Value" "680E"
 			(at 223.52 121.9199 0)
 			(effects
