File: boards/GIMIX DMA SASI/GIMIX DMA SASI_production/power.kicad_sch (KiCad schematic)
At the start: 53 parts, among them J1 Power, U1 7438, U10 74LS32, U11 74LS240, U13 74LS367, U15 7474, U16 74LS08, U17 7474, U18 74LS10, U19 74LS240, U2 74LS08, U20 74LS136, U21 74LS136, U22 74LS136, U23 74LS136, U24 74LS136, U3 74LS74, U33 LM7805_TO220, U34 LM7805_TO220, U35 74LS244, U36 74LS244, U38 LM7805_TO220, U4 74LS74, U5 74LS20, U6 7438, U7 7438, U8 7438, U9 7438

Commit message: DMA SASI update
Parts:
- R6: value ? -> 470E
Changed lines of the file:
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@@
 		(title "GIMIX DMA SASI Controller")
 		(date "2026-06-15")
-		(rev "0.4")
+		(rev "0.5")
 		(company "100% Offner")
-		(comment 1 "v0.1: Initial")
-		(comment 2 "v0.2: cleanup for production, gerbers exported")
+		(comment 1 "v0.4: add BlueSCSI v2 Mounting Holes, rotate 50p conn., add Logic Anlyzer Pins")
+		(comment 2 "v0.5: Resistor Values and more Testpoints added")
 	)
 	(junction
@@
 			)
 		)
-		(property "Value" "?"
+		(property "Value" "470E"
 			(at 275.59 27.9399 0)
 			(effects
