File: boards/GIMIX DMA SASI/GIMIX DMA SASI_production/sasi.kicad_sch (KiCad schematic)
At the start: 19 parts, among them J2 SASI, U1 7438, U10 74LS32, U11 74LS240, U15 7474, U16 74LS08, U17 7474, U18 74LS10, U19 74LS240, U29 74LS273, U30 74LS273, U31 74LS240, U32 74LS244, U6 7438, U7 7438, U8 7438, U9 7438

Commit message: SASI rework for BlueSCSI
Parts:
- added H1, H2, H3: MountingHole, MountingHole:MountingHole_3.2mm_M3_ISO14580, symbol Mechanical:MountingHole
- added J3: Conn_01x20, Connector_PinHeader_2.54mm:PinHeader_1x20_P2.54mm_Vertical, symbol Connector_Generic:Conn_01x20
- J2: footprint Connector_PinHeader_2.54mm:PinHeader_2x25_P2.54mm_Vertical -> Connector_PinHeader_2.54mm:PinHeader_2x25_P2.54mm_Horizontal
Connections:
- net GND: now also J3.10 (Pin_10), J3.11 (Pin_11), J3.12 (Pin_12), J3.9 (Pin_9)
- net ~{ACK}: now also J3.14 (Pin_14)
- net ~{BUSY}: now also J3.13 (Pin_13)
- net ~{C/D}: now also J3.18 (Pin_18)
- net ~{I/O}: now also J3.20 (Pin_20)
- net ~{MSG}: now also J3.16 (Pin_16)
- net ~{REQ}: now also J3.19 (Pin_19)
- net ~{SD0}: now also J3.1 (Pin_1)
- net ~{SD1}: now also J3.2 (Pin_2)
- net ~{SD2}: now also J3.3 (Pin_3)
- net ~{SD3}: now also J3.4 (Pin_4)
- net ~{SD4}: now also J3.5 (Pin_5)
- net ~{SD5}: now also J3.6 (Pin_6)
- net ~{SD6}: now also J3.7 (Pin_7)
- net ~{SD7}: now also J3.8 (Pin_8)
- net ~{SEL}: now also J3.17 (Pin_17)
- net ~{SRST}: now also J3.15 (Pin_15)

Commit message: DMA SASI update
Parts:
- added TP1: SASIR, Connector_PinHeader_2.54mm:PinHeader_1x01_P2.54mm_Vertical, symbol Connector:TestPoint
- added TP2: SASIW, Connector_PinHeader_2.54mm:PinHeader_1x01_P2.54mm_Vertical, symbol Connector:TestPoint
- added TP3: WE, Connector_PinHeader_2.54mm:PinHeader_1x01_P2.54mm_Vertical, symbol Connector:TestPoint
- added TP4: RE, Connector_PinHeader_2.54mm:PinHeader_1x01_P2.54mm_Vertical, symbol Connector:TestPoint
- added TP5: OutputBuffer On, Connector_PinHeader_2.54mm:PinHeader_1x01_P2.54mm_Vertical, symbol Connector:TestPoint
- added TP6: StatusBuffer On, Connector_PinHeader_2.54mm:PinHeader_1x01_P2.54mm_Vertical, symbol Connector:TestPoint
- J3: value Conn_01x20 -> Debug
- R7: value ? -> 1k
Connections:
- net ~{RE}: now also TP4.1
- net ~{SASIR}: now also TP1.1
- net ~{SASIW}: now also TP2.1
- net ~{WE}: now also TP3.1
- net at U15.12 (D), U15.5 (Q), U7.10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: now also TP6.1
- net at U17.5 (Q), U6.1, U7.1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: now also TP5.1
