File: boards/GIMIX DMA SASI/GIMIX DMA SASI_production/switches.kicad_sch (KiCad schematic)
At the start: 15 parts, among them SW1 SW_DIP_x10, SW2 SW_DIP_x10, U10 74LS32, U11 74LS240, U20 74LS136, U21 74LS136, U22 74LS136, U23 74LS136, U24 74LS136

Commit message: DMA SASI update
Parts:
- R1: value ? -> 10E
- R2, R5: value ? -> 680E
- RP1, RP2: value ? -> 10k
Changed lines of the file:
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@@
 		(title "GIMIX DMA SASI Controller")
 		(date "2026-06-15")
-		(rev "0.4")
+		(rev "0.5")
 		(company "100% Offner")
-		(comment 1 "v0.1: Initial")
-		(comment 2 "v0.2: cleanup for production, gerbers exported")
+		(comment 1 "v0.4: add BlueSCSI v2 Mounting Holes, rotate 50p conn., add Logic Anlyzer Pins")
+		(comment 2 "v0.5: Resistor Values and more Testpoints added")
 	)
 	(text "DMA extended Address enable"
@@
 			)
 		)
-		(property "Value" "?"
+		(property "Value" "10k"
 			(at 95.758 103.378 0)
 			(effects
@@
 			)
 		)
-		(property "Value" "?"
+		(property "Value" "10E"
 			(at 148.59 136.398 90)
 			(effects
@@
 			)
 		)
-		(property "Value" "?"
+		(property "Value" "680E"
 			(at 154.94 135.8899 0)
 			(effects
@@
 			)
 		)
-		(property "Value" "?"
+		(property "Value" "10k"
 			(at 97.028 77.978 0)
 			(effects
@@
 			)
 		)
-		(property "Value" "?"
+		(property "Value" "680E"
 			(at 118.11 138.4299 0)
 			(effects
